Commit message: List of TODO on readme

File: smart2_description/urdf/create_1.urdf.xacro (robot description, xacro)
@@ -1,8 +1,8 @@
 <?xml version="1.0" ?>
 <robot name="create_1" xmlns:xacro="http://ros.org/wiki/xacro">
-  <xacro:include filename="$(find ca_description)/urdf/create_base.urdf.xacro" />
-  <xacro:include filename="$(find ca_description)/urdf/create_1_gazebo.urdf.xacro" />
+  <xacro:include filename="$(find smart2_description)/urdf/create_base.urdf.xacro" />
+  <xacro:include filename="$(find smart2_description)/urdf/create_1_gazebo.urdf.xacro" />
   <xacro:create_base wheel_separation="0.26" base_diameter="0.3302">
-    <mesh filename="package://ca_description/meshes/create_1.dae" />
+    <mesh filename="package://smart2_description/meshes/smart_2.dae" />
   </xacro:create_base>
 </robot>

File: smart2_description/urdf/create_base.urdf.xacro (robot description, xacro)
@@ -30,5 +30,5 @@
   </xacro:macro>
   <xacro:macro name="create_base" params="diffdrive_update_rate:=40 wheel_separation wheel_radius:=0.036 wheel_width:=0.024 wheel_torque:=1.0 wheel_accel:=1.8 mass_kg:=3.5 base_diameter *mesh">
-    <xacro:include filename="$(find ca_description)/urdf/create_base_gazebo.urdf.xacro" />
+    <xacro:include filename="$(find smart2_description)/urdf/create_base_gazebo.urdf.xacro" />
     <link name="base_footprint">
     <visual>

Commit message: adjusted size of robot model .dae, improved position of camera_link and base_scan frames and created an rviz file

File: smart2_description/urdf/create_1.urdf.xacro (robot description, xacro)
@@ -4,5 +4,5 @@
   <xacro:include filename="$(find smart2_description)/urdf/create_1_gazebo.urdf.xacro" />
   <xacro:create_base wheel_separation="0.26" base_diameter="0.3302">
-    <mesh filename="package://smart2_description/meshes/smart_2.dae" />
+    <mesh filename="package://smart2_description/meshes/smart_2_resize.dae" />
   </xacro:create_base>
 </robot>
